File: drone.kicad_pcb (KiCad board)
At the start: 2 copper layers, 76 x 76 mm, 75 parts, among them IC1 TP4056-42-ESOP8, J2 USB_C_Receptacle_USB2.0_16P, J3 Conn_01x02_Socket, J6 Conn_01x02_Socket, J7 Conn_01x02_Socket, J8 Conn_01x02_Socket, Q1 AO3401A, Q2 SI2302DS, Q3 SI2302DS, Q4 SI2302DS, Q6 SI2302DS, SW2 SK12D07VG4, U1 ESP32-WROOM-32, U2 DDC114TU-7-F1, U3 CH340C, U4 MPU-6050, U5 MIC5219-3.3YM5

Commit message: finalize
Parts:
- moved C1 3.00 mm to (154.0, 164.9)
- moved C2 3.00 mm to (151.0, 164.9)
Routing:
- net +BATT: track 348.9 -> 350.5 mm
Changed lines of the file:
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@@
 	(footprint "Capacitor_SMD:C_0603_1608Metric"
 		(layer "B.Cu")
-		(at 151 164.9)
+		(at 154 164.9)
 		(descr "Capacitor SMD 0603 (1608 Metric), square (rectangular) end terminal, IPC-7351 nominal, (Body size source: IPC-SM-782 page 76, https://www.pcb-3d.com/wordpress/wp-content/uploads/ipc-sm-782a_amendment_1_and_2.pdf), generated with kicad-footprint-generator")
 		(tags "capacitor")
@@
 	(footprint "Capacitor_SMD:C_0603_1608Metric"
 		(layer "B.Cu")
-		(at 154 164.9)
+		(at 151 164.9)
 		(descr "Capacitor SMD 0603 (1608 Metric), square (rectangular) end terminal, IPC-7351 nominal, (Body size source: IPC-SM-782 page 76, https://www.pcb-3d.com/wordpress/wp-content/uploads/ipc-sm-782a_amendment_1_and_2.pdf), generated with kicad-footprint-generator")
 		(tags "capacitor")
@@
 	(segment
 		(start 160.0721 154.397)
-		(end 152.4788 146.8037)
+		(end 152.4788 145.7537)
 		(width 1.3)
 		(layer "F.Cu")
@@
 	)
 	(segment
-		(start 118.1038 146.8037)
+		(start 118.1038 145.7537)
 		(end 116.3397 148.5678)
 		(width 1.3)
@@
 	)
 	(segment
-		(start 152.4788 146.8037)
-		(end 118.1038 146.8037)
+		(start 152.4788 145.7537)
+		(end 118.1038 145.7537)
 		(width 1.34)
 		(layer "F.Cu")
